File: embedded-system/embedded-system.kicad_sch (KiCad schematic)
At the start: 7 parts, among them M1 Motor_Servo, M2 Motor_Servo

Commit message: feat: added schematic for embedded systems
Designed a basic PCB for the embedded system
Parts:
- RV1, RV2: footprint (none) -> custom-footprint:p103
Changed lines of the file:
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@@
 			)
 		)
-		(property "Footprint" ""
+		(property "Footprint" "custom-footprint:p103"
 			(at 115.57 73.66 0)
 			(effects
@@
 			)
 		)
-		(property "Footprint" ""
+		(property "Footprint" "custom-footprint:p103"
 			(at 115.57 86.36 0)
 			(effects
