File: embedded-pcb/embedded-pcb.kicad_sch (KiCad schematic)
At the start: 8 parts

Commit message: feat: small update to schematic
Parts:
- added A2: Arduino_Nano_v2.x, Module:Arduino_Nano, symbol MCU_Module:Arduino_Nano_v2.x
- added M1: Motor_Servo, symbol Motor:Motor_Servo
- added RV3: R_Potentiometer_Trim, Potentiometer_THT:Potentiometer_ACP_CA9-H2,5_Horizontal, symbol Device:R_Potentiometer_Trim
Connections:
- new net: A2.29 (GND), RV3.1
- new net: A2.19 (A0), RV3.2
- new net: A2.17 (3V3), RV3.3
- new net: A2.13 (D10), M1.1 (PWM)
- new net: A2.27 (+5V), M1.2 (+)
- new net: A2.4 (GND), M1.3 (-)
