File: embedded-pcb/embedded-pcb.kicad_pcb (KiCad board)
At the start: 2 copper layers, 8 parts

Commit message: feat: optimised tracks
Parts:
- moved A1 86.5 mm to (97.1, 63.0), turned to 180 degrees
- moved R2 69.0 mm to (94.0, 45.7)
- moved R1 68.7 mm to (89.5, 43.2)
- moved Servos1 66.8 mm to (83.2, 73.5)
- moved D1 56.5 mm to (72.0, 61.2), turned to -90 degrees
- moved D2 43.5 mm to (72.0, 69.2), turned to -90 degrees
- moved RV2 36.8 mm to (74.5, 37.5)
- moved RV1 24.0 mm to (74.5, 49.5)
Routing:
- net /GND: track 146.6 -> 84.5 mm
- net /PWM: track 95.6 -> 74.2 mm
- net Net-(D2-A): track 19.6 -> 36.7 mm
- net Net-(D1-A): track 18.4 -> 31.1 mm
- net Net-(A1-A0): track 22.2 -> 9.92 mm
- net /Vcc: track 63.4 -> 56.3 mm
- net Net-(A1-D9): track 8.05 -> 3.16 mm
- net Net-(A1-D10): track 3.50 -> 7.65 mm
- net Net-(A1-A1): track 13.4 -> 14.7 mm
