File: Embedded Systems/embedded-system/embedded-system.kicad_sch (KiCad schematic)
At the start: 7 parts, among them M1 Motor_Servo, M2 Motor_Servo

Commit message: feat: updated schematic
Parts:
- added R1, R2: 200, symbol Device:R
Connections:
- net at D1.2 (A): now also R1.1; no longer A1.28 (D13)
- net at D2.2 (A): now also R2.1; no longer A1.27 (D12)
- new net: A1.28 (D13), R1.2
- new net: A1.27 (D12), R2.2
Other:
- note added: "Rev 1"
Changed lines of the file:
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@@
 		(comment 3 "Designed by Oskar Meszaros")
+	)
+	(text "Rev 1"
+		(exclude_from_sim no)
+		(at 115.57 100.076 0)
+		(effects
+			(font
+				(size 1.27 1.27)
+			)
+		)
 	)
 	(junction
@@
 	(wire
 		(pts
+			(xy 64.77 109.22) (xy 82.55 109.22)
+		)
+		(stroke
+			(width 0)
+			(type default)
+		)
+	)
+	(wire
+		(pts
 			(xy 104.14 77.47) (xy 104.14 90.17)
 		)
@@
 	(wire
 		(pts
+			(xy 82.55 95.25) (xy 104.14 95.25)
+		)
+		(stroke
+			(width 0)
+			(type default)
+		)
+	)
+	(wire
+		(pts
 			(xy 104.14 90.17) (xy 115.57 90.17)
 		)
@@
 	(wire
 		(pts
+			(xy 90.17 109.22) (xy 96.52 109.22)
+		)
+		(stroke
+			(width 0)
+			(type default)
+		)
+	)
+	(wire
+		(pts
+			(xy 66.04 99.06) (xy 82.55 99.06)
+		)
+		(stroke
+			(width 0)
+			(type default)
+		)
+	)
+	(wire
+		(pts
 			(xy 95.25 69.85) (xy 95.25 86.36)
 		)
@@
 	(wire
 		(pts
-			(xy 66.04 99.06) (xy 96.52 99.06)
-		)
-		(stroke
-			(width 0)
-			(type default)
-		)
-	)
-	(wire
-		(pts
 			(xy 105.41 60.96) (xy 105.41 48.26)
 		)
@@
 	(wire
 		(pts
-			(xy 64.77 109.22) (xy 96.52 109.22)
-		)
-		(stroke
-			(width 0)
-			(type default)
-		)
-	)
-	(wire
-		(pts
 			(xy 105.41 38.1) (xy 85.09 38.1)
 		)
@@
 	(wire
 		(pts
+			(xy 90.17 99.06) (xy 96.52 99.06)
+		)
+		(stroke
+			(width 0)
+			(type default)
+		)
+	)
+	(wire
+		(pts
 			(xy 111.76 73.66) (xy 96.52 73.66)
 		)
@@
 		)
 	)
-	(wire
-		(pts
-			(xy 104.14 95.25) (xy 82.55 95.25)
-		)
-		(stroke
-			(width 0)
-			(type default)
+	(symbol
+		(lib_id "Device:R")
+		(at 86.36 99.06 270)
+		(unit 1)
+		(exclude_from_sim no)
+		(in_bom yes)
+		(on_board yes)
+		(dnp no)
+		(property "Reference" "R1"
+			(at 86.36 94.234 90)
+			(effects
+				(font
+					(size 1.27 1.27)
+				)
+			)
+		)
+		(property "Value" "200"
+			(at 86.36 96.774 90)
+			(effects
+				(font
+					(size 1.27 1.27)
+				)
+			)
+		)
+		(property "Footprint" ""
+			(at 86.36 97.282 90)
+			(effects
+				(font
+					(size 1.27 1.27)
+				)
+				(hide yes)
+			)
+		)
+		(property "Datasheet" "~"
+			(at 86.36 99.06 0)
+			(effects
+				(font
+					(size 1.27 1.27)
+				)
+				(hide yes)
+			)
+		)
+		(property "Description" "Resistor"
+			(at 86.36 99.06 0)
+			(effects
+				(font
+					(size 1.27 1.27)
+				)
+				(hide yes)
+			)
+		)
+		(pin "2"
+		)
+		(pin "1"
+		)
+		(instances
+			(project ""
+				(path "/de6be016-d057-4e05-93ca-5815b4f6abac"
+					(reference "R1")
+					(unit 1)
+				)
+			)
 		)
 	)
@@
 					(unit 1)
 				)
+			)
+		)
+	)
+	(symbol
+		(lib_id "Device:R")
+		(at 86.36 109.22 270)
+		(unit 1)
+		(exclude_from_sim no)
+		(in_bom yes)
+		(on_board yes)
+		(dnp no)
+		(property "Reference" "R2"
+			(at 86.36 104.902 90)
+			(effects
+				(font
+					(size 1.27 1.27)
+				)
+			)
+		)
+		(property "Value" "200"
+			(at 86.36 106.934 90)
+			(effects
+				(font
+					(size 1.27 1.27)
+				)
+			)
+		)
+		(property "Footprint" ""
+			(at 86.36 107.442 90)
+			(effects
+				(font
+					(size 1.27 1.27)
+				)
+				(hide yes)
+			)
+		)
+		(property "Datasheet" "~"
+			(at 86.36 109.22 0)
+			(effects
+				(font
+					(size 1.27 1.27)
+				)
+				(hide yes)
+			)
+		)
+		(property "Description" "Resistor"
+			(at 86.36 109.22 0)
+			(effects
+				(font
+					(size 1.27 1.27)
+				)
+				(hide yes)
+			)
+		)
+		(pin "1"
+		)
+		(pin "2"
+		)
+		(instances
+			(project ""
+				(path "/de6be016-d057-4e05-93ca-5815b4f6abac"
+					(reference "R2")
+					(unit 1)
+				)

Commit message: feat: updated schematic
Parts:
- removed A1: Arduino_UNO_R3, Module:Arduino_UNO_R3, symbol MCU_Module:Arduino_UNO_R3
- removed R1, R2: 200, symbol Device:R
- added A1: Arduino_Nano_v3.x, Module:Arduino_Nano, symbol MCU_Module:Arduino_Nano_v3.x
- added R1, R2: 47, Resistor_THT:R_Axial_DIN0207_L6.3mm_D2.5mm_P10.16mm_Horizontal, symbol Device:R_Small_US
- added R3, R4: 1k, Resistor_THT:R_Axial_DIN0207_L6.3mm_D2.5mm_P10.16mm_Horizontal, symbol Device:R_Small_US
- added SW1: SW_DIP_x02, Button_Switch_THT:SW_DIP_SPSTx02_Piano_10.8x6.64mm_W7.62mm_P2.54mm, symbol Switch:SW_DIP_x02
- D1, D2: footprint LED_THT:LED_D5.0mm_Horizontal_O6.35mm_Z15.0mm -> LED_THT:LED_D5.0mm
- RV1, RV2: footprint custom-footprint:p103 -> Potentiometer_THT:Potentiometer_ACP_CA14-H5_Horizontal
Connections:
- net at D1.2 (A): now also R1.1
- net at M1.2 (+), M2.2 (+), RV1.1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: now also A1.17 (3V3), SW1.3, SW1.4
- net at RV1.2: now also A1.19 (A0)
- net at M2.1 (PWM): now also A1.10 (D7)
- net at M1.1 (PWM): now also A1.9 (D6)
- net at RV2.2: now also A1.20 (A1)
- net at D2.2 (A): now also R2.1
- new net: A1.4 (GND), M1.3 (-), M2.3 (-), R1.2, R2.2, R3.2, R4.2
- new net: A1.29 (GND), RV1.3, RV2.3
- new net: A1.5 (D2), D2.1 (K)
- new net: A1.6 (D3), D1.1 (K)
- new net: A1.7 (D4), R3.1, SW1.1
- new net: A1.8 (D5), R4.1, SW1.2
Other:
- note removed: "Rev 1"
